File: Archive/V3/Eagle/Iridium_9603_Beacon.sch (EAGLE design)
At the start: 79 parts, among them CON4 uFL, J1 SS4-10-3.50-X-D, Q1 DMG3415U-7, U1 MCP111T-240E/TT, U2 SPX3819-3.3, U3 LTC3225EDDB#TRMPBF, U4 MPL3115A2LGA8, U5 ATSAMD21G18_QFN, U6 MAX-M8, U7 LT1634-1,25BMCMS8, X1 32.768

Commit message: Initial update for V4 - still work in progress
Parts:
- removed C18: 10nF, microbuilder:CAP_CERAMIC0805-NOOUTLINE
- removed C19: 10uF, microbuilder:CAP_CERAMIC0805-NOOUTLINE
- removed CON4: uFL, microbuilder:ANTENNA_U.FL
- removed D4: MBR120, microbuilder:DIODE-SCHOTTKYSOD-123
- removed GND2, GND3, VBUS: (no value), adafruit:PINHD-1X1
- removed GNSS, IRIDIUM: SMA-142-0711-821/826, con-coax:SMA-142-0711-821/826
- removed JP2: JUMPER-PAD-3-2OF3_NC_BY_TRACE_LARGE, SparkFun-Passives:JUMPER-PAD-3-2OF3_NC_BY_TRACE_LARGE
- removed L1: 33nH, microbuilder:FERRITE-0805NO
- removed LED2: RED, microbuilder:LED0805_NOOUTLINE
- removed R10: 2.2K, microbuilder:RESISTOR_0603_NOOUT
- removed R11: 30K, microbuilder:RESISTOR0805_NOOUTLINE
- removed R9: 10 ohm, microbuilder:RESISTOR0805_NOOUTLINE
- removed U7: LT1634-1,25BMCMS8, linear-technology:LT1634-1,25BMCMS8
- added GND.: (no value), adafruit:PINHD-1X1
- BAT1, BAT2, BAT3: device SparkFun-Electromechanical:BATTERYKEYSTONE92 -> SparkFun-Electromechanical:BATTERYKEYSTONE82
- LED1: value (none) -> RED; device SparkFun-LED:WS2812B -> microbuilder:LED0805_NOOUTLINE
- R2: value 12K -> 30K
- R7: value 47k -> 2.2K
- U1: value MCP111T-240E/TT -> MCP111T-195I/TT; MPN MCP111T-240E/TT -> (none)
- U6: value MAX-M8 -> SAM-M8Q; device ubloxLib:MAX-M8 -> ubloxLib:SAM-M8Q
Connections:
- removed net GPS_ANT: GNSS.1, L1.P$2, U6.11_RF_IN
- removed net N$1 (its old number): C18.1, L1.P$1, R9.1
- removed net N$16: CON1.VBUS, D4.A
- removed net N$17: JP2.3, R2.2
- removed net N$18: JP2.1, R11.2
- removed net N$3 (its old number): LED2.A, R10.2
- removed net VCC_RF: R9.2, U6.14_VCC_RF
- net +3V3: now also U6.V_BCKP; no longer C19.1, LED1.VDD, U6.6_V_BCKP
- net 3V3SW: now also U6.VCC, U6.VCC_IO; no longer U6.7_VCC_IO, U6.8_VCC
- net A0: no longer R7.2, U7.VOUT
- net D0: now also U6.TXD; no longer U6.2_TXD
- net D1: now also U6.RXD; no longer U6.3_RXD
- net D13: now also R7.1; no longer LED1.DIN, R10.1
- net GND: now also GND..1, LED1.C, U6.GND; no longer C18.2, C19.2, CON4.GND@0, CON4.GND@1, GND2.1, GND3.1, GNSS.2, IRIDIUM.2, LED1.VSS, LED2.C, R11.1, U6.10_GND, U6.12_GND, U6.1_GND, U7.GND
- net N$11: now also R2.2; no longer JP2.2
- net N$2: now also LED1.A, R7.2; no longer CON4.SIGNAL, IRIDIUM.1
- net VBUS: now also CON1.VBUS; no longer D4.C, R7.1, VBUS.1
Other:
- note added: "3 x AAA Energiser Ultimate Lithium in Keystone Electronics 82 clips"
- note added: "LED"
- note added: "u-blox SAM-M8Q"
- note removed: "150mA"
- note removed: "3 x AA Energiser Ultimate Lithium in Keystone Electronics 92 clips"
- note removed: "60mA"
- note removed: "Iridium 9603 Beacon Notes"
- note removed: "LEDs"
- note removed: "Notes on power voltages: MBR120 diode has a forward voltage drop of approx.: 0.26V at 170mA 0.19V at 12mA MBR120 diode plus SPX3819-3.3 regulator have a combined voltage drop of approx.: 0.22V at 12mA; 0.36V at 170mA. Output starts to collapse when 'solar' voltage drops below approx.: 3.65V at 12mA; 3.80V at 170mA. Reported voltage on A7 will bottom out at 3.38V / 3.43V even though the actual vol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"
- note removed: "V4: Power: 3 x AA batteries in Keystone 92 clips GNSS: u-blox MAX-M8Q with SMA antenna SMA antenna for 9603N Added WS2812B LED Added LT1634-1,25BMCMS8 voltage reference to allow low battery voltages to be measured Added protection diode for USB power Added split pad to select supercapacitor charge current"
- note removed: "WS2812B"
- note removed: "u-blox MAX-M8Q"
