File: Archive/V4/Eagle/Iridium_9603_Beacon.brd (EAGLE design)
At the start: 57.6 x 66 mm, 100 parts, among them CON4 uFL, J1 SS4-10-3.50-X-D, Q1 DMG3415U-7, Q2 DMG3415U-7, Q3 DMG3415U-7, Q4 DMG3415U-7, Q5 2N2222, U1 MCP111T-240E/TT, U2 SPX3819-3.3, U3 LTC3225EDDB#TRMPBF, U4 MPL3115A2LGA8, U5 ATSAMD21G18_QFN, U6 MAX-M8, U7 LT1634-1,25BMCMS8, X1 32.768

Commit message: Major update for V5
Parts:
- removed BAT-, COM1, COM2, NC1, NC2, NO1, NO2, RST: (no value), adafruit:1X01
- removed D5, D6: MBR120, microbuilder:SOD-123
- removed Q2, Q3, Q4: DMG3415U-7, microbuilder:SOT23-WIDE
- removed Q5: 2N2222, transistor:SOT23-BEC
- removed R12, R13: 100K, microbuilder:0805-NO
- removed R14: 1K, microbuilder:0603-NO
- removed R15, R16, R17: 10K, microbuilder:0603-NO
- removed RELAY1: G6SK-2_DC5, G6SK-2_DC5:G6SK2DC5
- moved GND3 54.6 mm to (54.6, 16.2), turned to 270 degrees
- moved GND 53.7 mm to (3.81, 36.1), turned to 90 degrees
- moved SOLAR2+ 32.5 mm to (20.3, 63.5)
- moved SOLAR1+ 30.0 mm to (25.4, 63.5)
- moved SOLAR1- 23.1 mm to (32.2, 63.5)
- moved SOLAR2- 15.5 mm to (37.2, 63.5)
- moved D3 13.1 mm to (25.4, 57.2)
- moved D2 2.63 mm to (21.6, 57.1)
- moved D1 2.54 mm to (21.0, 53.1)
- moved FD2 2.54 mm to (52.5, 61.0)
- moved SWCLK 2.54 mm to (52.1, 18.7)
- moved SWDIO 2.54 mm to (54.6, 18.7)
- moved VBUS 2.54 mm to (52.1, 16.2)
- moved R1 1.99 mm to (19.9, 39.0), turned to 90 degrees
- moved R4 1.20 mm to (41.9, 40.0)
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- renumbered CS to SD_CS
Connections:
- removed net EXT_PWR: J1.1, J1.2, Q4.3
- removed net GNDA: CON4.1, CON4.2, IRIDIUM.G@1, IRIDIUM.G@2, IRIDIUM.G@3, IRIDIUM.G@4
- removed net N$15 (its old number): BAT-.1, BAT3.GND@1, BAT3.GND@2
- removed net N$19: Q4.1, Q5.C, R15.2
- removed net N$20: Q5.B, R14.2
- removed net N$23: NC1.1, RELAY1.3
- removed net N$24: COM1.1, RELAY1.4
- removed net N$25: NO1.1, RELAY1.5
- removed net N$26: NO2.1, RELAY1.8
- removed net N$27: COM2.1, RELAY1.9
- removed net N$28: NC2.1, RELAY1.10
- removed net RESET_RELAY: D3.C, Q3.3, RELAY1.6
- removed net SET_RELAY: D2.C, Q2.3, RELAY1.1
- net !RESET: no longer RST.1
- net +3V3: no longer Q2.2, Q3.2, R1.1, R12.2, R13.2
- net A3: now also J1.19; no longer J1.12
- net A5: no longer R14.1, R17.1
- net D2: no longer Q3.1, R13.1
- net D5: no longer R16.1
- net D7: no longer Q2.1, R12.1
- net GND: now also BAT3.GND@1, BAT3.GND@2, CON4.1, CON4.2, IRIDIUM.G@1, IRIDIUM.G@2, IRIDIUM.G@3, IRIDIUM.G@4, R1.1; no longer D2.A, D3.A, Q5.E, R16.2, R17.2, RELAY1.12, RELAY1.7
- net LTC3225_VOUT: now also J1.1, J1.2; no longer Q4.2, R15.1
- net N$14: now also D2.A; no longer D5.A
- net N$4: now also D3.A; no longer D6.A
- net VBUS: now also D2.C, D3.C; no longer D5.C, D6.C
Routing:
- net N$19: track 38.4 -> 0.00 mm, vias 2 -> 0
- net D7: track 34.7 -> 0.00 mm, vias 2 -> 0
- net D2: track 26.2 -> 0.00 mm, vias 4 -> 0
- net !RESET: track 57.4 -> 34.8 mm, vias 5 -> 4
- net N$15 (its old number): track 18.2 -> 0.00 mm
- net LTC3225_VOUT: track 22.1 -> 38.4 mm
- net RESET_RELAY: track 13.9 -> 0.00 mm
- net N$25: track 13.8 -> 0.00 mm
- net N$24: track 12.0 -> 0.00 mm
- net N$23: track 11.0 -> 0.00 mm
- net +3V3: track 195.2 -> 184.2 mm
- net EXT_PWR: track 9.50 -> 0.00 mm
- net GND: track 692.6 -> 700.0 mm, vias 17 -> 15
- net A5: track 5.58 -> 0.00 mm
- net SET_RELAY: track 5.51 -> 0.00 mm
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- removed copper zone on layer 1, net GNDA
- removed copper zone on layer 16, net GNDA
Other:
- board text added: "150mA"
- board text added: "5.3V"
- board text added: "5.5V Max"
- board text added: "Iridium 9603N Beacon V4"
- board text removed: "150"
- board text removed: "30VDC 2A MAX"
- board text removed: "5.3 V"
- board text removed: "5.5V MAX"
- board text removed: "GND"
- board text removed: "Iridium 9603N Beacon V5"
- board text removed: "mA"
