File: Archive/V4/Eagle/Iridium_9603_Beacon.sch (EAGLE design)
At the start: 100 parts, among them CON4 uFL, J1 SS4-10-3.50-X-D, Q1 DMG3415U-7, Q2 DMG3415U-7, Q3 DMG3415U-7, Q4 DMG3415U-7, Q5 2N2222, U1 MCP111T-240E/TT, U2 SPX3819-3.3, U3 LTC3225EDDB#TRMPBF, U4 MPL3115A2LGA8, U5 ATSAMD21G18_QFN, U6 MAX-M8, U7 LT1634-1,25BMCMS8, X1 32.768

Commit message: Major update for V5
Parts:
- removed BAT-, COM1, COM2, NC1, NC2, NO1, NO2, RST: (no value), adafruit:PINHD-1X1
- removed D5, D6: MBR120, microbuilder:DIODE-SCHOTTKYSOD-123
- removed Q2, Q3, Q4: DMG3415U-7, microbuilder:MOSFET-PWIDE
- removed Q5: 2N2222, transistor:MMBT2222ALT1-NPN-SOT23-BEC
- removed R12, R13: 100K, microbuilder:RESISTOR0805_NOOUTLINE
- removed R14: 1K, microbuilder:RESISTOR_0603_NOOUT
- removed R15, R16, R17: 10K, microbuilder:RESISTOR_0603_NOOUT
- removed RELAY1: G6SK-2_DC5, G6SK-2_DC5:G6SK-2_DC5
- renumbered CS to SD_CS
Connections:
- removed net EXT_PWR: J1.1, J1.2, Q4.D
- removed net GNDA: CON4.GND@0, CON4.GND@1, IRIDIUM.2
- removed net N$15 (its old number): BAT-.1, BAT3.-
- removed net N$19: Q4.G, Q5.C, R15.2
- removed net N$20: Q5.B, R14.2
- removed net N$23: NC1.1, RELAY1.NC(1)
- removed net N$24: COM1.1, RELAY1.COM(1)
- removed net N$25: NO1.1, RELAY1.NO(1)
- removed net N$26: NO2.1, RELAY1.NO(2)
- removed net N$27: COM2.1, RELAY1.COM(2)
- removed net N$28: NC2.1, RELAY1.NC(2)
- removed net RESET_RELAY: D3.C, Q3.D, RELAY1.COIL2+
- removed net SET_RELAY: D2.C, Q2.D, RELAY1.COIL1+
- net !RESET: no longer RST.1
- net +3V3: no longer Q2.S, Q3.S, R1.1, R12.2, R13.2
- net A3: now also J1.19; no longer J1.12
- net A5: no longer R14.1, R17.1
- net D2: no longer Q3.G, R13.1
- net D5: no longer R16.1
- net D7: no longer Q2.G, R12.1
- net GND: now also BAT3.-, CON4.GND@0, CON4.GND@1, IRIDIUM.2, R1.1; no longer D2.A, D3.A, Q5.E, R16.2, R17.2, RELAY1.COIL1-, RELAY1.COIL2-
- net LTC3225_VOUT: now also J1.1, J1.2; no longer Q4.S, R15.1
- net N$14: now also D2.A; no longer D5.A
- net N$4: now also D3.A; no longer D6.A
- net VBUS: now also D2.C, D3.C; no longer D5.C, D6.C
Other:
- note added: "Notes on power voltages: MBR120 diode has a forward voltage drop of approx.: 0.26V at 170mA 0.19V at 12mA MBR120 diode plus SPX3819-3.3 regulator have a combined voltage drop of approx.: 0.22V at 12mA; 0.36V at 170mA. Output starts to collapse when 'solar' voltage drops below approx.: 3.65V at 12mA; 3.80V at 170mA. Reported voltage on A7 will bottom out at 3.38V / 3.43V even though the actual vol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"
- note added: "See Page 6 for Change Log"
- note removed: "Cut link if installing power switch"
- note removed: "Notes on power voltages: MBR120 diode has a forward voltage drop of approx.: 0.19V at 12mA 0.26V at 170mA MBR120 diode plus SPX3819-3.3 regulator have a combined voltage drop of approx.: 0.22V at 12mA 0.36V at 170mA Regulator output starts to collapse when 'solar' voltage drops below approx.: 3.65V at 12mA; 3.80V at 170mA. Reported voltage on A7 will bottom out at 3.38V / 3.43V even though the ac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"
- note removed: "Omron G6SK-2 3VDC"
- note removed: "Pads for battery power switch"
- note removed: "See Page 7 for Change Log"
- note removed: "V5: Added a dual coil latching DPDT relay (Omron G6SK-2 3VDC; enabled via D2 and D7) Solar pins have been moved to make room for the relay Isolated the Iridium antenna ground 9603N EXT_PWR is now switched via Q4 and Q5 (enabled via A5/D19) Added a pull-down resistor for LTC3225 ~SHDN R1 now pulls up (not down) A3 now connects to 9603N Ring Indicator (not Network Available) Added a pad for an exte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"
